File: HW/RT_STACK.kicad_pcb (KiCad board)
At the start: 6 copper layers, 150 x 150 mm, 475 parts, among them IC1 IFX007TAUMA1, IC10 IFX007TAUMA1, IC11 IFX007TAUMA1, IC12 IFX007TAUMA1, IC2 IFX007TAUMA1, IC3 IFX007TAUMA1, IC4 IFX007TAUMA1, IC5 IFX007TAUMA1, IC6 IFX007TAUMA1, IC7 IFX007TAUMA1, IC8 IFX007TAUMA1, IC9 IFX007TAUMA1, J1 5601381861, J11 Conn_02x03_Odd_Even, J12 Conn_02x03_Odd_Even, J2 Conn_02x18_Odd_Even, J3 Conn_02x10_Odd_Even, J4 Conn_02x10_Odd_Even, J5 Conn_02x20_Odd_Even, J6 Conn_02x10_Odd_Even, J7 Conn_02x10_Odd_Even, J8 Conn_02x07_Odd_Even, J9 Conn_02x15_Odd_Even, Q1 SUD80460E, Q10 SUD80460E, Q11 SUD80460E, Q12 SUD80460E, Q13 SUD80460E, Q14 SUD80460E, Q15 SUD80460E, Q16 SUD80460E, Q17 SUD80460E, Q18 SUD80460E, Q19 RGPR30BM40, Q2 SUD80460E, Q20 RGPR30BM40, Q21 RGPR30BM40, Q22 RGPR30BM40, Q23 RGPR30BM40, Q24 RGPR30BM40, Q25 RGPR30BM40, Q26 RGPR30BM40, Q27 RGPR30BM40, Q28 RGPR30BM40, Q29 RGPR30BM40, Q3 SUD80460E, Q30 RGPR30BM40, Q31 BUK9230-100B, Q32 BUK9230-100B, Q33 SS8550, Q34 STD30NF06LT4, Q35 SS8550, Q36 STD30NF06LT4, Q4 SUD80460E, Q5 SUD80460E, Q6 SUD80460E, Q7 SUD80460E, Q8 SUD80460E, Q9 SUD80460E, U1 SN74AHC1G02DCKR, U10 SN74AHC1G08DCKR, U11 SN74AHC1G08DCKR, U12 SN74AHC1G08DCKR, U13 SN74AHC1G02DCKR, U14 SN74AHC1G02DCKR, U15 SN74AHC1G08DCKR, U16 SN74AHC1G08DCKR, U17 SN74AHC1G08DCKR, U18 SN74AHC1G08DCKR, U19 IR2101, U2 SN74AHC1G02DCKR, U20 IR2101, U21 ACS722xLCTR-20AB, U22 ACS722xLCTR-20AB, U23 TC4427xOA, U24 IR2101, U25 IR2101, U26 ACS722xLCTR-20AB, U27 ACS722xLCTR-20AB, U28 TC4427xOA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

Commit message: Ver2
Second HW rev + SW update
Parts:
- added C122: 47p, Capacitor_SMD:C_0402_1005Metric, F.Cu at (112.1, 39.9)
- added C123: 47p, Capacitor_SMD:C_0402_1005Metric, F.Cu at (112.1, 43.7)
- added C124: 100n, Capacitor_SMD:C_0402_1005Metric, F.Cu at (101.1, 42.4)
- added H10: MountingHole_Pad, MountingHole:MountingHole_2.2mm_M2_DIN965_Pad_TopBottom, F.Cu at (155.9, 88.2)
- added H11: MountingHole_Pad, MountingHole:MountingHole_2.2mm_M2_DIN965_Pad_TopBottom, F.Cu at (169.8, 88.2)
- added J10: LD09S13A4GX00LF, iota:LD09S13A4GX00LF, F.Cu at (78.6, 43.0)
- added JP4: Jumper_2_Open, Jumper:SolderJumper-2_P1.3mm_Open_RoundedPad1.0x1.5mm, F.Cu at (112.1, 37.3)
- added R168: 60, Resistor_SMD:R_0402_1005Metric, F.Cu at (109.1, 37.3)
- added U55: TJA1051T-3, Package_SO:SOIC-8_3.9x4.9mm_P1.27mm, F.Cu at (106.6, 41.8)
- moved G*** 12.7 mm to (32.7, 35.1), turned to 30 degrees
Connections:
- J9 pad 27: PA11 -> CAN1_L
- J9 pad 28: PA12 -> CAN1_H
- U41 pad 72: PA11 -> /MCU/CAN_TX
- U41 pad 73: PA12 -> /MCU/CAN_RX
Routing:
- net /MCU/CAN_RX: track 0.00 -> 79.2 mm, vias 0 -> 2
- net /MCU/CAN_TX: track 0.00 -> 78.4 mm, vias 0 -> 2
- net PA12: track 74.4 -> 0.00 mm, vias 1 -> 0
- net VBUS: track 466.7 -> 536.7 mm
- net PA11: track 66.1 -> 0.00 mm, vias 1 -> 0
- net CAN1_L: track 0.00 -> 52.1 mm
- net CAN1_H: track 0.00 -> 47.3 mm
- net +5V: track 64.4 -> 67.0 mm, vias 35 -> 36
- net Net-(JP4-A): track 0.00 -> 1.87 mm
- net GND: track 20.8 -> 22.3 mm, vias 54 -> 55
- net +3.3V: track 148.4 -> 149.8 mm, vias 44 -> 45
Other:
- board text added: "COMP7_IN CANH PA9 PA15 PD0 PF0 PF1 PD1 PC15 PB9 PB7 PB5 PB3 PD6 PD4"
- board text added: "GND CANL COMP7_OUT PE7 PF2 PG10 PF10 PF9 PC14 PB8 PB6 PB4 PD7 PD5 PD3"
- board text removed: "COMP7_IN PA12 PA9 PA15 PD0 PF0 PF1 PD1 PC15 PB9 PB7 PB5 PB3 PD6 PD4"
- board text removed: "GND PA11 COMP7_OUT PE7 PF2 PG10 PF10 PF9 PC14 PB8 PB6 PB4 PD7 PD5 PD3"
