File: HW/RT_STACK.kicad_pcb (KiCad board)
At the start: 6 copper layers, 150 x 150 mm, 484 parts, among them IC1 IFX007TAUMA1, IC10 IFX007TAUMA1, IC11 IFX007TAUMA1, IC12 IFX007TAUMA1, IC2 IFX007TAUMA1, IC3 IFX007TAUMA1, IC4 IFX007TAUMA1, IC5 IFX007TAUMA1, IC6 IFX007TAUMA1, IC7 IFX007TAUMA1, IC8 IFX007TAUMA1, IC9 IFX007TAUMA1, J1 5601381861, J10 LD09S13A4GX00LF, J11 Conn_02x03_Odd_Even, J12 Conn_02x03_Odd_Even, J2 Conn_02x18_Odd_Even, J3 Conn_02x10_Odd_Even, J4 Conn_02x10_Odd_Even, J5 Conn_02x20_Odd_Even, J6 Conn_02x10_Odd_Even, J7 Conn_02x10_Odd_Even, J8 Conn_02x07_Odd_Even, J9 Conn_02x15_Odd_Even, Q1 SUD80460E, Q10 SUD80460E, Q11 SUD80460E, Q12 SUD80460E, Q13 SUD80460E, Q14 SUD80460E, Q15 SUD80460E, Q16 SUD80460E, Q17 SUD80460E, Q18 SUD80460E, Q19 RGPR30BM40, Q2 SUD80460E, Q20 RGPR30BM40, Q21 RGPR30BM40, Q22 RGPR30BM40, Q23 RGPR30BM40, Q24 RGPR30BM40, Q25 RGPR30BM40, Q26 RGPR30BM40, Q27 RGPR30BM40, Q28 RGPR30BM40, Q29 RGPR30BM40, Q3 SUD80460E, Q30 RGPR30BM40, Q31 BUK9230-100B, Q32 BUK9230-100B, Q33 SS8550, Q34 STD30NF06LT4, Q35 SS8550, Q36 STD30NF06LT4, Q4 SUD80460E, Q5 SUD80460E, Q6 SUD80460E, Q7 SUD80460E, Q8 SUD80460E, Q9 SUD80460E, U1 SN74AHC1G02DCKR, U10 SN74AHC1G08DCKR, U11 SN74AHC1G08DCKR, U12 SN74AHC1G08DCKR, U13 SN74AHC1G02DCKR, U14 SN74AHC1G02DCKR, U15 SN74AHC1G08DCKR, U16 SN74AHC1G08DCKR, U17 SN74AHC1G08DCKR, U18 SN74AHC1G08DCKR, U19 IR2101, U2 SN74AHC1G02DCKR, U20 IR2101, U21 ACS722xLCTR-20AB, U22 ACS722xLCTR-20AB, U23 TC4427xOA, U24 IR2101, U25 IR2101, U26 ACS722xLCTR-20AB, U27 ACS722xLCTR-20AB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

Commit message: v0.2 BOM
Other:
- board text added: "V0.2"
- board text removed: "V0.1"
Changed lines of the file:
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@@
 			(outputformat 1)
 			(mirror no)
-			(drillshape 1)
+			(drillshape 0)
 			(scaleselection 1)
-			(outputdirectory "")
+			(outputdirectory "../FAB/")
 		)
 	)
@@
 		)
 	)
-	(gr_text "V0.1"
+	(gr_text "V0.2"
 		(at 159.65 122.5 0)
 		(layer "F.SilkS")
@@
 			)
 		)
+	)
+	(dimension
+		(type orthogonal)
+		(layer "F.SilkS")
+		(pts
+			(xy 175.7 180) (xy 175.7 30.025)
+		)
+		(height 9.8)
+		(orientation 1)
+		(format
+			(prefix "")
+			(suffix "")
+			(units 3)
+			(units_format 0)
+			(precision 4)
+			(suppress_zeroes yes)
+		)
+		(style
+			(thickness 0.1)
+			(arrow_length 1.27)
+			(text_position_mode 0)
+			(arrow_direction outward)
+			(extension_height 0.58642)
+			(extension_offset 0.5)
+			(keep_text_aligned yes)
+		)
+		(gr_text "149.975"
+			(at 184.4 105.0125 90)
+			(layer "F.SilkS")
+			(effects
+				(font
+					(size 1 1)
+					(thickness 0.1)
+				)
+			)
+		)
+	)
+	(dimension
+		(type orthogonal)
+		(layer "F.SilkS")
+		(pts
+			(xy 30 176) (xy 180 176)
+		)
+		(height 12)
+		(orientation 0)
+		(format
+			(prefix "")
+			(suffix "")
+			(units 3)
+			(units_format 0)
+			(precision 4)
+			(suppress_zeroes yes)
+		)
+		(style
+			(thickness 0.1)
+			(arrow_length 1.27)
+			(text_position_mode 0)
+			(arrow_direction outward)
+			(extension_height 0.58642)
+			(extension_offset 0.5)
+			(keep_text_aligned yes)
+		)
+		(gr_text "150"
+			(at 105 186.9 0)
+			(layer "F.SilkS")
+			(effects
+				(font
+					(size 1 1)
+					(thickness 0.1)
+				)
+			)
+		)
