File: HW/RT_STACK.kicad_sch (KiCad schematic)
At the start: 9 parts

Commit message: Ver2
Second HW rev + SW update
Parts:
- added H10, H11: MountingHole_Pad, MountingHole:MountingHole_2.2mm_M2_DIN965_Pad_TopBottom, symbol Mechanical:MountingHole_Pad
Connections:
- new net +BATT: H10.1, H11.1
