File: HW/conn.kicad_sch (KiCad schematic)
At the start: 11 parts, among them J1 5601381861, J11 Conn_02x03_Odd_Even, J12 Conn_02x03_Odd_Even, J2 Conn_02x18_Odd_Even, J3 Conn_02x10_Odd_Even, J4 Conn_02x10_Odd_Even, J5 Conn_02x20_Odd_Even, J6 Conn_02x10_Odd_Even, J7 Conn_02x10_Odd_Even, J8 Conn_02x07_Odd_Even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

Commit message: Ver2
Second HW rev + SW update
Parts:
- added J10: LD09S13A4GX00LF, iota:LD09S13A4GX00LF, symbol iota:LD09S13A4GX00LF
Connections:
- net GND: now also J10.10 (MH1), J10.11 (MH2), J10.3, J10.5, J10.6
- net PA11: now also J10.2
- net PA12: now also J10.7
- no-connect marks 0 -> 4
